Commit message: Gazebo files

File: slam/dekutamr_description/urdf/materials.xacro (robot description, xacro)
@@ -1,6 +1,12 @@
 <?xml version="1.0" ?>
 <robot name="dekutamr" xmlns:xacro="http://www.ros.org/wiki/xacro" >
-<material name="silver">
-  <color rgba="0.700 0.700 0.700 1.000"/>
-</material>
+  <material name="silver">
+    <color rgba="0.700 0.700 0.700 1.000"/>
+  </material>
+  <material name="blue">
+    <color rgba="0.000 0.000 1.000 1.000"/>
+  </material>
+  <material name="green">
+    <color rgba="0.000 1.000 0.000 1.000"/>
+  </material>
 </robot>
