Commit message: base_link -> base footprint

File: slam/dekutamr_description/urdf/dekutamr.xacro (robot description, xacro)
@@ -1,180 +1,195 @@
 <?xml version="1.0" ?>
 <robot name="dekutamr" xmlns:xacro="http://www.ros.org/wiki/xacro">
-<xacro:include filename="$(find dekutamr_description)/urdf/materials.xacro" />
-<xacro:include filename="$(find dekutamr_description)/urdf/dekutamr.trans" />
-<xacro:include filename="$(find dekutamr_description)/urdf/dekutamr.gazebo" />
-<link name="base_link">
-  <inertial>
-    <origin xyz="0.1402992667578377 0.0 0.10323362010897062" rpy="0 0 0"/>
-    <mass value="59.838037523886456"/>
-    <inertia ixx="0.297515" iyy="0.462372" izz="0.562002" ixy="0.0" iyz="0.0" ixz="-3e-06"/>
-  </inertial>
-  <visual>
-    <origin xyz="0 0 0" rpy="0 0 0"/>
-    <geometry>
-      <mesh filename="file://$(find dekutamr_description)/meshes/base_link.stl" scale="0.001 0.001 0.001"/>
-    </geometry>
-    <material name="silver"/>
-  </visual>
-  <collision>
-    <origin xyz="0 0 0" rpy="0 0 0"/>
-    <geometry>
-      <mesh filename="file://$(find dekutamr_description)/meshes/base_link.stl" scale="0.001 0.001 0.001"/>
-    </geometry>
-  </collision>
-</link>
-<link name="frwheel_link_1">
-  <inertial>
-    <origin xyz="5.551115123125783e-17 -0.01050464503450281 0.0" rpy="0 0 0"/>
-    <mass value="1.3803967660818925"/>
-    <inertia ixx="0.000734" iyy="0.001247" izz="0.000734" ixy="-0.0" iyz="-0.0" ixz="0.0"/>
-  </inertial>
-  <visual>
-    <origin xyz="-0.21339 0.109 -0.0425" rpy="0 0 0"/>
-    <geometry>
-      <mesh filename="file://$(find dekutamr_description)/meshes/frwheel_link_1.stl" scale="0.001 0.001 0.001"/>
-    </geometry>
-    <material name="silver"/>
-  </visual>
-  <collision>
-    <origin xyz="-0.21339 0.109 -0.0425" rpy="0 0 0"/>
-    <geometry>
-      <mesh filename="file://$(find dekutamr_description)/meshes/frwheel_link_1.stl" scale="0.001 0.001 0.001"/>
-    </geometry>
-  </collision>
-</link>
-<link name="flwheel_link_1">
-  <inertial>
-    <origin xyz="5.551115123125783e-17 0.010504645034502769 0.0" rpy="0 0 0"/>
-    <mass value="1.3803967660818925"/>
-    <inertia ixx="0.000734" iyy="0.001247" izz="0.000734" ixy="0.0" iyz="0.0" ixz="0.0"/>
-  </inertial>
-  <visual>
-    <origin xyz="-0.21339 -0.109 -0.0425" rpy="0 0 0"/>
-    <geometry>
-      <mesh filename="file://$(find dekutamr_description)/meshes/flwheel_link_1.stl" scale="0.001 0.001 0.001"/>
-    </geometry>
-    <material name="silver"/>
-  </visual>
-  <collision>
-    <origin xyz="-0.21339 -0.109 -0.0425" rpy="0 0 0"/>
-    <geometry>
-      <mesh filename="file://$(find dekutamr_description)/meshes/flwheel_link_1.stl" scale="0.001 0.001 0.001"/>
-    </geometry>
-  </collision>
-</link>
-<link name="blwheel_link_1">
-  <inertial>
-    <origin xyz="6.938893903907228e-17 0.010504645034502769 -1.3877787807814457e-17" rpy="0 0 0"/>
-    <mass value="1.3803967660818925"/>
-    <inertia ixx="0.000734" iyy="0.001247" izz="0.000734" ixy="0.0" iyz="-0.0" ixz="-0.0"/>
-  </inertial>
-  <visual>
-    <origin xyz="-0.0425 -0.109 -0.0425" rpy="0 0 0"/>
-    <geometry>
-      <mesh filename="file://$(find dekutamr_description)/meshes/blwheel_link_1.stl" scale="0.001 0.001 0.001"/>
-    </geometry>
-    <material name="silver"/>
-  </visual>
-  <collision>
-    <origin xyz="-0.0425 -0.109 -0.0425" rpy="0 0 0"/>
-    <geometry>
-      <mesh filename="file://$(find dekutamr_description)/meshes/blwheel_link_1.stl" scale="0.001 0.001 0.001"/>
-    </geometry>
-  </collision>
-</link>
-<link name="brwheel_link_1">
-  <inertial>
-    <origin xyz="6.938893903907228e-17 -0.01050464503450281 -1.3877787807814457e-17" rpy="0 0 0"/>
-    <mass value="1.3803967660818925"/>
-    <inertia ixx="0.000734" iyy="0.001247" izz="0.000734" ixy="-0.0" iyz="-0.0" ixz="-0.0"/>
-  </inertial>
-  <visual>
-    <origin xyz="-0.0425 0.109 -0.0425" rpy="0 0 0"/>
-    <geometry>
-      <mesh filename="file://$(find dekutamr_description)/meshes/brwheel_link_1.stl" scale="0.001 0.001 0.001"/>
-    </geometry>
-    <material name="silver"/>
-  </visual>
-  <collision>
-    <origin xyz="-0.0425 0.109 -0.0425" rpy="0 0 0"/>
-    <geometry>
-      <mesh filename="file://$(find dekutamr_description)/meshes/brwheel_link_1.stl" scale="0.001 0.001 0.001"/>
-    </geometry>
-  </collision>
-</link>
-<link name="lidar_llink_1">
-  <inertial>
-    <origin xyz="2.7755575615628914e-17 6.391374769427968e-18 0.011555000000000037" rpy="0 0 0"/>
-    <mass value="0.6981609656059645"/>
-    <inertia ixx="0.000245" iyy="0.000245" izz="0.000428" ixy="0.0" iyz="0.0" ixz="0.0"/>
-  </inertial>
-  <visual>
-    <origin xyz="-0.1403 -0.0 -0.19709" rpy="0 0 0"/>
-    <geometry>
-      <mesh filename="file://$(find dekutamr_description)/meshes/lidar_llink_1.stl" scale="0.001 0.001 0.001"/>
-    </geometry>
-    <material name="silver"/>
-  </visual>
-  <collision>
-    <origin xyz="-0.1403 -0.0 -0.19709" rpy="0 0 0"/>
-    <geometry>
-      <mesh filename="file://$(find dekutamr_description)/meshes/lidar_llink_1.stl" scale="0.001 0.001 0.001"/>
-    </geometry>
-  </collision>
-</link>
-<link name="camera_link_1">
-  <inertial>
-    <origin xyz="0.001879766284094475 7.140431765511469e-14 0.0005413220291505816" rpy="0 0 0"/>
-    <mass value="0.04675581383016766"/>
-    <inertia ixx="1.6e-05" iyy="3e-06" izz="1.3e-05" ixy="0.0" iyz="-0.0" ixz="-0.0"/>
-  </inertial>
-  <visual>
-    <origin xyz="-0.19494 -0.0 -0.18709" rpy="0 0 0"/>
-    <geometry>
-      <mesh filename="file://$(find dekutamr_description)/meshes/camera_link_1.stl" scale="0.001 0.001 0.001"/>
-    </geometry>
-    <material name="silver"/>
-  </visual>
-  <collision>
-    <origin xyz="-0.19494 -0.0 -0.18709" rpy="0 0 0"/>
-    <geometry>
-      <mesh filename="file://$(find dekutamr_description)/meshes/camera_link_1.stl" scale="0.001 0.001 0.001"/>
-    </geometry>
-  </collision>
-</link>
-<joint name="fr_joint" type="continuous">
-  <origin xyz="0.21339 -0.109 0.0425" rpy="0 0 0"/>
-  <parent link="base_link"/>
-  <child link="frwheel_link_1"/>
-  <axis xyz="0.0 -1.0 0.0"/>
-</joint>
-<joint name="fl_joint" type="continuous">
-  <origin xyz="0.21339 0.109 0.0425" rpy="0 0 0"/>
-  <parent link="base_link"/>
-  <child link="flwheel_link_1"/>
-  <axis xyz="0.0 1.0 0.0"/>
-</joint>
-<joint name="bl_joint" type="continuous">
-  <origin xyz="0.0425 0.109 0.0425" rpy="0 0 0"/>
-  <parent link="base_link"/>
-  <child link="blwheel_link_1"/>
-  <axis xyz="0.0 1.0 0.0"/>
-</joint>
-<joint name="br_joint" type="continuous">
-  <origin xyz="0.0425 -0.109 0.0425" rpy="0 0 0"/>
-  <parent link="base_link"/>
-  <child link="brwheel_link_1"/>
-  <axis xyz="0.0 -1.0 0.0"/>
-</joint>
-<joint name="lidar_joint" type="fixed">
-  <origin xyz="0.1403 0.0 0.19709" rpy="0 0 0"/>
-  <parent link="base_link"/>
-  <child link="lidar_llink_1"/>
-</joint>
-<joint name="camera_joint" type="fixed">
-  <origin xyz="0.19494 0.0 0.18709" rpy="0 0 0"/>
-  <parent link="base_link"/>
-  <child link="camera_link_1"/>
-</joint>
+  <xacro:include filename="$(find dekutamr_description)/urdf/materials.xacro" />
+  <xacro:include filename="$(find dekutamr_description)/urdf/dekutamr.trans" />
+  <xacro:include filename="$(find dekutamr_description)/urdf/dekutamr.gazebo" />
+  <!-- Base footprint at origin -->
+  <link name="base_footprint"/>
+  <joint name="base_footprint_to_base_link" type="fixed">
+    <parent link="base_footprint"/>
+    <child link="base_link"/>
+    <origin xyz="-0.007 0 0" rpy="0 0 0"/>
+  </joint>
+  <link name="base_link">
+    <inertial>
+      <origin xyz="0 0 0.10323362010897062" rpy="0 0 0"/>
+      <mass value="59.838037523886456"/>
+      <inertia ixx="0.297515" iyy="0.462372" izz="0.562002" ixy="0.0" iyz="0.0" ixz="-3e-06"/>
+    </inertial>
+    <visual>
+      <origin xyz="0 0 0" rpy="0 0 0"/>
+      <geometry>
+        <mesh filename="file://$(find dekutamr_description)/meshes/base_link.stl" scale="0.001 0.001 0.001"/>
+      </geometry>
+      <material name="silver"/>
+    </visual>
+    <collision>
+      <origin xyz="0 0 0" rpy="0 0 0"/>
+      <geometry>
+        <mesh filename="file://$(find dekutamr_description)/meshes/base_link.stl" scale="0.001 0.001 0.001"/>
+      </geometry>
+    </collision>
+  </link>
+  <!-- Front Right Wheel -->
+  <link name="frwheel_link_1">
+    <inertial>
+      <origin xyz="0.003 -0.01050464503450281 0.0" rpy="0 0 0"/>
+      <mass value="1.3803967660818925"/>
+      <inertia ixx="0.000734" iyy="0.001247" izz="0.000734" ixy="0" iyz="0" ixz="0"/>
+    </inertial>
+    <visual>
+      <origin xyz="-0.21039 0.109 -0.0425" rpy="0 0 0"/>
+      <geometry>
+        <mesh filename="file://$(find dekutamr_description)/meshes/frwheel_link_1.stl" scale="0.001 0.001 0.001"/>
+      </geometry>
+      <material name="silver"/>
+    </visual>
+    <collision>
+      <origin xyz="-0.21039 0.109 -0.0425" rpy="0 0 0"/>
+      <geometry>
+        <mesh filename="file://$(find dekutamr_description)/meshes/frwheel_link_1.stl" scale="0.001 0.001 0.001"/>
+      </geometry>
+    </collision>
+  </link>
+  <!-- Front Left Wheel -->
+  <link name="flwheel_link_1">
+    <inertial>
+      <origin xyz="0.003 0.010504645034502769 0.0" rpy="0 0 0"/>
+      <mass value="1.3803967660818925"/>
+      <inertia ixx="0.000734" iyy="0.001247" izz="0.000734" ixy="0" iyz="0" ixz="0"/>
+    </inertial>
+    <visual>
+      <origin xyz="-0.21039 -0.109 -0.0425" rpy="0 0 0"/>
+      <geometry>
+        <mesh filename="file://$(find dekutamr_description)/meshes/flwheel_link_1.stl" scale="0.001 0.001 0.001"/>
+      </geometry>
+      <material name="silver"/>
+    </visual>
+    <collision>
+      <origin xyz="-0.21039 -0.109 -0.0425" rpy="0 0 0"/>
+      <geometry>
+        <mesh filename="file://$(find dekutamr_description)/meshes/flwheel_link_1.stl" scale="0.001 0.001 0.001"/>
+      </geometry>
+    </collision>
+  </link>
+  <!-- Back Left Wheel -->
+  <link name="blwheel_link_1">
+    <inertial>
+      <origin xyz="0.003 0.010504645034502769 0.0" rpy="0 0 0"/>
+      <mass value="1.3803967660818925"/>
+      <inertia ixx="0.000734" iyy="0.001247" izz="0.000734" ixy="0" iyz="0" ixz="0"/>
+    </inertial>
+    <visual>
+      <origin xyz="-0.0395 -0.109 -0.0425" rpy="0 0 0"/>
+      <geometry>
+        <mesh filename="file://$(find dekutamr_description)/meshes/blwheel_link_1.stl" scale="0.001 0.001 0.001"/>
+      </geometry>
+      <material name="silver"/>
+    </visual>
+    <collision>
+      <origin xyz="-0.0395 -0.109 -0.0425" rpy="0 0 0"/>
+      <geometry>
+        <mesh filename="file://$(find dekutamr_description)/meshes/blwheel_link_1.stl" scale="0.001 0.001 0.001"/>
+      </geometry>
+    </collision>
+  </link>
+  <!-- Back Right Wheel -->
+  <link name="brwheel_link_1">
+    <inertial>
+      <origin xyz="0.003 -0.01050464503450281 0.0" rpy="0 0 0"/>
+      <mass value="1.3803967660818925"/>
+      <inertia ixx="0.000734" iyy="0.001247" izz="0.000734" ixy="0" iyz="0" ixz="0"/>
+    </inertial>
+    <visual>
+      <origin xyz="-0.0395 0.109 -0.0425" rpy="0 0 0"/>
+      <geometry>
+        <mesh filename="file://$(find dekutamr_description)/meshes/brwheel_link_1.stl" scale="0.001 0.001 0.001"/>
+      </geometry>
+      <material name="silver"/>
+    </visual>
+    <collision>
+      <origin xyz="-0.0395 0.109 -0.0425" rpy="0 0 0"/>
+      <geometry>
+        <mesh filename="file://$(find dekutamr_description)/meshes/brwheel_link_1.stl" scale="0.001 0.001 0.001"/>
+      </geometry>
+    </collision>
+  </link>
+  <!-- Joints remain unchanged -->
+  <joint name="fr_joint" type="continuous">
+    <origin xyz="0.08009 -0.109 0.0425" rpy="0 0 0"/>
+    <parent link="base_link"/>
+    <child link="frwheel_link_1"/>
+    <axis xyz="0 -1 0"/>
+  </joint>
+  <joint name="fl_joint" type="continuous">
+    <origin xyz="0.08009 0.109 0.0425" rpy="0 0 0"/>
+    <parent link="base_link"/>
+    <child link="flwheel_link_1"/>
+    <axis xyz="0 1 0"/>
+  </joint>
+  <joint name="bl_joint" type="continuous">
+    <origin xyz="-0.1048 0.109 0.0425" rpy="0 0 0"/>
+    <parent link="base_link"/>
+    <child link="blwheel_link_1"/>
+    <axis xyz="0 1 0"/>
+  </joint>
+  <joint name="br_joint" type="continuous">
+    <origin xyz="-0.1048 -0.109 0.0425" rpy="0 0 0"/>
+    <parent link="base_link"/>
+    <child link="brwheel_link_1"/>
+    <axis xyz="0 -1 0"/>
+  </joint>
+  <!-- Lidar Link -->
+  <link name="lidar_llink_1">
+    <inertial>
+      <origin xyz="0.003 0 0.011555" rpy="0 0 0"/>
+      <mass value="0.69816"/>
+      <inertia ixx="0.000245" iyy="0.000245" izz="0.000428" ixy="0" iyz="0" ixz="0"/>
+    </inertial>
+    <visual>
+      <origin xyz="-0.1373 0 -0.19709" rpy="0 0 0"/>
+      <geometry>
+        <mesh filename="file://$(find dekutamr_description)/meshes/lidar_llink_1.stl" scale="0.001 0.001 0.001"/>
+      </geometry>
+      <material name="silver"/>
+    </visual>
+    <collision>
+      <origin xyz="-0.1373 0 -0.19709" rpy="0 0 0"/>
+      <geometry>
+        <mesh filename="file://$(find dekutamr_description)/meshes/lidar_llink_1.stl" scale="0.001 0.001 0.001"/>
+      </geometry>
+    </collision>
+  </link>
+  <!-- Camera Link -->
+  <link name="camera_link_1">
+    <inertial>
+      <origin xyz="0.003 0 0.000541" rpy="0 0 0"/>
+      <mass value="0.04676"/>
+      <inertia ixx="1.6e-05" iyy="3e-06" izz="1.3e-05" ixy="0" iyz="0" ixz="0"/>
+    </inertial>
+    <visual>
+      <origin xyz="-0.19194 0 -0.18709" rpy="0 0 0"/>
+      <geometry>
+        <mesh filename="file://$(find dekutamr_description)/meshes/camera_link_1.stl" scale="0.001 0.001 0.001"/>
+      </geometry>
+      <material name="silver"/>
+    </visual>
+    <collision>
+      <origin xyz="-0.19194 0 -0.18709" rpy="0 0 0"/>
+      <geometry>
+        <mesh filename="file://$(find dekutamr_description)/meshes/camera_link_1.stl" scale="0.001 0.001 0.001"/>
+      </geometry>
+    </collision>
+  </link>
+  <!-- Sensor joints remain unchanged -->
+  <joint name="lidar_joint" type="fixed">
+    <origin xyz="0.007 0 0.19709" rpy="0 0 0"/>
+    <parent link="base_link"/>
+    <child link="lidar_llink_1"/>
+  </joint>
+  <joint name="camera_joint" type="fixed">
+    <origin xyz="0.06164 0 0.18709" rpy="0 0 0"/>
+    <parent link="base_link"/>
+    <child link="camera_link_1"/>
+  </joint>
 </robot>

File: slam/dekutamr_description/urdf/materials.xacro (robot description, xacro)
@@ -1,12 +1,6 @@
 <?xml version="1.0" ?>
 <robot name="dekutamr" xmlns:xacro="http://www.ros.org/wiki/xacro" >
-  <material name="silver">
-    <color rgba="0.700 0.700 0.700 1.000"/>
-  </material>
-  <material name="blue">
-    <color rgba="0.000 0.000 1.000 1.000"/>
-  </material>
-  <material name="green">
-    <color rgba="0.000 1.000 0.000 1.000"/>
-  </material>
+<material name="silver">
+  <color rgba="0.700 0.700 0.700 1.000"/>
+</material>
 </robot>
